Commit message: Replacing aubo_iS20 to aubo_iS20L

File: aubo_description/urdf/aubo_iS20L_21_calibrated.urdf (robot description, URDF)
Before this commit: robot aubo_iS20_T0, 8 links, 7 joints
Links:
- link base_link: geometry collision mesh filename=package://aubo_description/meshes/aubo_iS20L_21/collision/l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; visual mesh filename=package://aubo_description/meshes/aubo_iS20L_21/visual/link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
- link foreArm_Link: mass 7.099652 -> 6.748493; geometry collision mesh filename=package://aubo_description/meshes/aubo_iS20L_21/collision/l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; visual mesh filename=package://aubo_description/meshes/aubo_iS20L_21/visual/link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
- link shoulder_Link: geometry collision mesh filename=package://aubo_description/meshes/aubo_iS20L_21/collision/l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; visual mesh filename=package://aubo_description/meshes/aubo_iS20L_21/visual/link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
- link upperArm_Link: geometry collision mesh filename=package://aubo_description/meshes/aubo_iS20L_21/collision/l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; visual mesh filename=package://aubo_description/meshes/aubo_iS20L_21/visual/link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
- link wrist1_Link: mass 3.257300 -> 2.890610; geometry collision mesh filename=package://aubo_description/meshes/aubo_iS20L_21/collision/l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; visual mesh filename=package://aubo_description/meshes/aubo_iS20L_21/visual/link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
- link wrist2_Link: mass 3.257300 -> 2.890610; geometry collision mesh filename=package://aubo_description/meshes/aubo_iS20L_21/collision/l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; visual mesh filename=package://aubo_description/meshes/aubo_iS20L_21/visual/link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
- link wrist3_Link: geometry collision mesh filename=package://aubo_description/meshes/aubo_iS20L_21/collision/l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; visual mesh filename=package://aubo_description/meshes/aubo_iS20L_21/visual/link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
Joints:
- joint foreArm_joint: limit lower=-6.283185307179586476925286766559 upper=6.283185307179586476925286766559 effort=281 velocity=3.1104 -> lower=-6.283185307179586476925286766559 upper=6.283185307179586476925286766559 effort=267 velocity=4.14
- joint shoulder_joint: limit lower=-6.283185307179586476925286766559 upper=6.283185307179586476925286766559 effort=819 velocity=1.62 -> lower=-6.283185307179586476925286766559 upper=6.283185307179586476925286766559 effort=809 velocity=1.62
- joint upperArm_joint: limit lower=-6.283185307179586476925286766559 upper=6.283185307179586476925286766559 effort=819 velocity=1.62 -> lower=-6.283185307179586476925286766559 upper=6.283185307179586476925286766559 effort=809 velocity=1.62; origin xyz=-0.000638600 0.211336083 -0.000084467 rpy=-3.1415926535896399 -1.5703966468016928 1.5707963267947433 -> xyz=-0.000638600 0.209336083 -0.000083667 rpy=-3.1415926535896399 -1.5703966468016928 1.5707963267947433
- joint wrist1_joint: limit lower=-6.283185307179586476925286766559 upper=6.283185307179586476925286766559 effort=64 velocity=4.1469 -> lower=-6.283185307179586476925286766559 upper=6.283185307179586476925286766559 effort=58 velocity=5.1714105736592; origin xyz=0.826692800 -0.000001671 0.000663898 rpy=-3.1415926535897931 -0.0025167600251733 1.5707963267948966 -> xyz=0.825692800 -0.000001671 0.000663898 rpy=-3.1415926535897931 -0.0025167600251733 1.5707963267948966
- joint wrist2_joint: limit lower=-6.283185307179586476925286766559 upper=6.283185307179586476925286766559 effort=64 velocity=4.1469 -> lower=-6.283185307179586476925286766559 upper=6.283185307179586476925286766559 effort=58 velocity=5.1714105736592; origin xyz=-0.000348300 0.126497898 -0.000020975 rpy=-1.5709621367885287 -0.0000000000000000 0.0000000000000000 -> xyz=-0.000348300 0.124497898 -0.000020643 rpy=-1.5709621367885287 -0.0000000000000000 0.0000000000000000
- joint wrist3_joint: limit lower=-6.283185307179586476925286766559 upper=6.283185307179586476925286766559 effort=64 velocity=4.1469 -> lower=-6.283185307179586476925286766559 upper=6.283185307179586476925286766559 effort=58 velocity=3.1105; origin xyz=-0.000459700 -0.110298642 0.000547303 rpy=1.5658343569983284 -0.0000000000000000 0.0000000000000000 -> xyz=-0.000459700 -0.109298655 0.000542341 rpy=1.5658343569983284 -0.0000000000000000 0.0000000000000000
